Commit message: wheel collision corrected

File: urdf/robot.urdf (robot description, URDF)
Before this commit: robot kobuki, 4 links, 3 joints
Links:
- link wheel_l: geometry collision sphere radius=0.0352; visual mesh filename=package://kobuki_x360controller/meshes/wheel.stl
- link wheel_r: geometry collision sphere radius=0.0352; visual mesh filename=package://kobuki_x360controller/meshes/wheel.stl
Joints:
- joint j_wheel_l: limit (none) -> effort=1000.0 velocity=$(eval 1.0/0.0352); origin xyz=0 0.115 0 rpy=1.57079 0 0 -> xyz=0 0.115 0 rpy=$(eval pi/2) 0 0
- joint j_wheel_r: limit (none) -> effort=1000.0 velocity=$(eval 1.0/0.0352); origin xyz=0 -0.115 0 rpy=1.57079 0 0 -> xyz=0 -0.115 0 rpy=$(eval pi/2) 0 0

Commit message: Joints corrected

File: urdf/robot.urdf (robot description, URDF)
Before this commit: robot kobuki, 4 links, 3 joints
Links:
- removed link wheel_l
- removed link wheel_r
- added link left_wheel, mass 0.084; collision sphere radius=0.0352; visual mesh filename=package://kobuki_x360controller/meshes/wheel.stl
- added link right_wheel, mass 0.084; collision sphere radius=0.0352; visual mesh filename=package://kobuki_x360controller/meshes/wheel.stl
Joints:
- removed joint j_wheel_l
- removed joint j_wheel_r
- added joint left_wheel_joint: type continuous, parent chasis, child left_wheel, origin xyz=0 0.115 0 rpy=$(eval pi/2) 0 0, axis 0 0 1, limit effort=1000.0 velocity=$(eval 1.0/0.0352)
- added joint right_wheel_joint: type continuous, parent chasis, child right_wheel, origin xyz=0 -0.115 0 rpy=$(eval pi/2) 0 0, axis 0 0 1, limit effort=1000.0 velocity=$(eval 1.0/0.0352)
- joint fixed_joint: origin xyz=0.0 0.0 0.0 rpy=0.0 0.0 0.0 -> xyz=0.0 0.0 0.0352 rpy=0.0 0.0 0.0

Commit message: Output=screen python files

File: urdf/robot.urdf (robot description, URDF)
Before this commit: robot kobuki, 4 links, 3 joints
Joints:
- joint left_wheel_joint: limit effort=1000.0 velocity=$(eval 1.0/0.0352) -> effort=1000.0 velocity=${1.0/0.0352}; origin xyz=0 0.115 0 rpy=$(eval pi/2) 0 0 -> xyz=0 0.115 0 rpy=${pi/2} 0 0
- joint right_wheel_joint: limit effort=1000.0 velocity=$(eval 1.0/0.0352) -> effort=1000.0 velocity=${1.0/0.0352}; origin xyz=0 -0.115 0 rpy=$(eval pi/2) 0 0 -> xyz=0 -0.115 0 rpy=${pi/2} 0 0

Commit message: meshes modified; kinematics, controller and urdf corrected

File: urdf/robot.urdf (robot description, URDF)
Before this commit: robot kobuki, 4 links, 3 joints
Joints:
- joint left_wheel_joint: limit effort=1000.0 velocity=${1.0/0.0352} -> (none)
- joint right_wheel_joint: limit effort=1000.0 velocity=${1.0/0.0352} -> (none)
